File: hardware/kicad/enku-mainboard-r0.1/power.kicad_sch (KiCad schematic)
At the start: 34 parts

Commit message: Add R0.1 power bring-up test points
Parts:
- added TP_3V3: 3V3_SYS, TestPoint:TestPoint_Pad_D1.5mm, symbol ENKU:TESTPOINT
- added TP_GND_PWR: GND, TestPoint:TestPoint_Pad_D1.5mm, symbol ENKU:TESTPOINT
- added TP_REG_PG: REG_PG, TestPoint:TestPoint_Pad_D1.5mm, symbol ENKU:TESTPOINT
- added TP_SYS_EN: SYS_EN, TestPoint:TestPoint_Pad_D1.5mm, symbol ENKU:TESTPOINT
- added TP_VBAT: VBAT, TestPoint:TestPoint_Pad_D1.5mm, symbol ENKU:TESTPOINT
- added TP_VBUS_DOCK: VBUS_DOCK, TestPoint:TestPoint_Pad_D1.5mm, symbol ENKU:TESTPOINT
- added TP_VBUS_USB: VBUS_USB, TestPoint:TestPoint_Pad_D1.5mm, symbol ENKU:TESTPOINT
- added TP_VSYS: VSYS, TestPoint:TestPoint_Pad_D1.5mm, symbol ENKU:TESTPOINT
Connections:
- net 3V3_SYS: now also TP_3V3.1 (TP)
- net GND: now also TP_GND_PWR.1 (TP)
- net REG_PG: now also TP_REG_PG.1 (TP)
- net SYS_EN: now also TP_SYS_EN.1 (TP)
- net VBAT: now also TP_VBAT.1 (TP)
- net VBUS_DOCK: now also TP_VBUS_DOCK.1 (TP)
- net VBUS_USB: now also TP_VBUS_USB.1 (TP)
- net VSYS: now also TP_VSYS.1 (TP)
Changed lines of the file:
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@@
 	(text "TPS63802 replaces TPS63031 for first-spin headroom: 2A @ 3.3V for VIN>=2.3V, MODE low for power-save, 0.47uH DFE201612E-R47M=P2, 511k/91k feedback, 10uF input and 2x22uF output." (exclude_from_sim no) (at 25 30 0) (effects (font (size 1.05 1.05)) (justify left bottom)))
 	(text "R_MUX_ILIM=100k is a conservative R0.1 placeholder current-limit population; verify simultaneous source and inrush behavior on bench before production freeze." (exclude_from_sim no) (at 25 35 0) (effects (font (size 1.05 1.05)) (justify left bottom)))
+	(symbol (lib_id "ENKU:TESTPOINT") (at 35 180 0) (unit 1) (exclude_from_sim no) (in_bom yes) (on_board yes) (dnp no)
+		(property "Reference" "TP_GND_PWR" (at 35 177.46 0) (effects (font (size 0.9 0.9))))
+		(property "Value" "GND" (at 35 182.54 0) (effects (font (size 0.9 0.9))))
+		(property "Footprint" "TestPoint:TestPoint_Pad_D1.5mm" (at 35 180 0) (effects (font (size 0.9 0.9)) (hide yes)))
+		(property "Datasheet" "~" (at 35 180 0) (effects (font (size 0.9 0.9)) (hide yes)))
+		(property "Description" "ENKU R0.1 bring-up test point" (at 35 180 0) (effects (font (size 0.9 0.9)) (hide yes)))
+		(pin "1")
+		(instances (project "enku-mainboard-r0.1" (path "/10000000-0000-4000-8000-000000000001/10000000-0000-4000-8000-000000000010" (reference "TP_GND_PWR") (unit 1))))
+	)
+	(global_label "GND" (shape bidirectional) (at 31.19 180 0)
+		(effects (font (size 0.9 0.9)) (justify right bottom))
+)
+	(symbol (lib_id "ENKU:TESTPOINT") (at 65 180 0) (unit 1) (exclude_from_sim no) (in_bom yes) (on_board yes) (dnp no)
+		(property "Reference" "TP_VBUS_USB" (at 65 177.46 0) (effects (font (size 0.9 0.9))))
+		(property "Value" "VBUS_USB" (at 65 182.54 0) (effects (font (size 0.9 0.9))))
+		(property "Footprint" "TestPoint:TestPoint_Pad_D1.5mm" (at 65 180 0) (effects (font (size 0.9 0.9)) (hide yes)))
+		(property "Datasheet" "~" (at 65 180 0) (effects (font (size 0.9 0.9)) (hide yes)))
+		(property "Description" "ENKU R0.1 bring-up test point" (at 65 180 0) (effects (font (size 0.9 0.9)) (hide yes)))
+		(pin "1")
+		(instances (project "enku-mainboard-r0.1" (path "/10000000-0000-4000-8000-000000000001/10000000-0000-4000-8000-000000000010" (reference "TP_VBUS_USB") (unit 1))))
+	)
+	(global_label "VBUS_USB" (shape bidirectional) (at 61.19 180 0)
+		(effects (font (size 0.9 0.9)) (justify right bottom))
+)
+	(symbol (lib_id "ENKU:TESTPOINT") (at 95 180 0) (unit 1) (exclude_from_sim no) (in_bom yes) (on_board yes) (dnp no)
+		(property "Reference" "TP_VBUS_DOCK" (at 95 177.46 0) (effects (font (size 0.9 0.9))))
+		(property "Value" "VBUS_DOCK" (at 95 182.54 0) (effects (font (size 0.9 0.9))))
+		(property "Footprint" "TestPoint:TestPoint_Pad_D1.5mm" (at 95 180 0) (effects (font (size 0.9 0.9)) (hide yes)))
+		(property "Datasheet" "~" (at 95 180 0) (effects (font (size 0.9 0.9)) (hide yes)))
+		(property "Description" "ENKU R0.1 bring-up test point" (at 95 180 0) (effects (font (size 0.9 0.9)) (hide yes)))
+		(pin "1")
+		(instances (project "enku-mainboard-r0.1" (path "/10000000-0000-4000-8000-000000000001/10000000-0000-4000-8000-000000000010" (reference "TP_VBUS_DOCK") (unit 1))))
+	)
+	(global_label "VBUS_DOCK" (shape bidirectional) (at 91.19 180 0)
+		(effects (font (size 0.9 0.9)) (justify right bottom))
+)
+	(symbol (lib_id "ENKU:TESTPOINT") (at 125 180 0) (unit 1) (exclude_from_sim no) (in_bom yes) (on_board yes) (dnp no)
+		(property "Reference" "TP_VBAT" (at 125 177.46 0) (effects (font (size 0.9 0.9))))
+		(property "Value" "VBAT" (at 125 182.54 0) (effects (font (size 0.9 0.9))))
+		(property "Footprint" "TestPoint:TestPoint_Pad_D1.5mm" (at 125 180 0) (effects (font (size 0.9 0.9)) (hide yes)))
+		(property "Datasheet" "~" (at 125 180 0) (effects (font (size 0.9 0.9)) (hide yes)))
+		(property "Description" "ENKU R0.1 bring-up test point" (at 125 180 0) (effects (font (size 0.9 0.9)) (hide yes)))
+		(pin "1")
+		(instances (project "enku-mainboard-r0.1" (path "/10000000-0000-4000-8000-000000000001/10000000-0000-4000-8000-000000000010" (reference "TP_VBAT") (unit 1))))
+	)
+	(global_label "VBAT" (shape bidirectional) (at 121.19 180 0)
+		(effects (font (size 0.9 0.9)) (justify right bottom))
+)
+	(symbol (lib_id "ENKU:TESTPOINT") (at 155 180 0) (unit 1) (exclude_from_sim no) (in_bom yes) (on_board yes) (dnp no)
+		(property "Reference" "TP_VSYS" (at 155 177.46 0) (effects (font (size 0.9 0.9))))
+		(property "Value" "VSYS" (at 155 182.54 0) (effects (font (size 0.9 0.9))))
+		(property "Footprint" "TestPoint:TestPoint_Pad_D1.5mm" (at 155 180 0) (effects (font (size 0.9 0.9)) (hide yes)))
+		(property "Datasheet" "~" (at 155 180 0) (effects (font (size 0.9 0.9)) (hide yes)))
+		(property "Description" "ENKU R0.1 bring-up test point" (at 155 180 0) (effects (font (size 0.9 0.9)) (hide yes)))
+		(pin "1")
+		(instances (project "enku-mainboard-r0.1" (path "/10000000-0000-4000-8000-000000000001/10000000-0000-4000-8000-000000000010" (reference "TP_VSYS") (unit 1))))
+	)
+	(global_label "VSYS" (shape bidirectional) (at 151.19 180 0)
+		(effects (font (size 0.9 0.9)) (justify right bottom))
+)
+	(symbol (lib_id "ENKU:TESTPOINT") (at 185 180 0) (unit 1) (exclude_from_sim no) (in_bom yes) (on_board yes) (dnp no)
+		(property "Reference" "TP_3V3" (at 185 177.46 0) (effects (font (size 0.9 0.9))))
+		(property "Value" "3V3_SYS" (at 185 182.54 0) (effects (font (size 0.9 0.9))))
+		(property "Footprint" "TestPoint:TestPoint_Pad_D1.5mm" (at 185 180 0) (effects (font (size 0.9 0.9)) (hide yes)))
+		(property "Datasheet" "~" (at 185 180 0) (effects (font (size 0.9 0.9)) (hide yes)))
+		(property "Description" "ENKU R0.1 bring-up test point" (at 185 180 0) (effects (font (size 0.9 0.9)) (hide yes)))
+		(pin "1")
+		(instances (project "enku-mainboard-r0.1" (path "/10000000-0000-4000-8000-000000000001/10000000-0000-4000-8000-000000000010" (reference "TP_3V3") (unit 1))))
+	)
+	(global_label "3V3_SYS" (shape bidirectional) (at 181.19 180 0)
+		(effects (font (size 0.9 0.9)) (justify right bottom))
+)
+	(symbol (lib_id "ENKU:TESTPOINT") (at 215 180 0) (unit 1) (exclude_from_sim no) (in_bom yes) (on_board yes) (dnp no)
+		(property "Reference" "TP_SYS_EN" (at 215 177.46 0) (effects (font (size 0.9 0.9))))
+		(property "Value" "SYS_EN" (at 215 182.54 0) (effects (font (size 0.9 0.9))))
+		(property "Footprint" "TestPoint:TestPoint_Pad_D1.5mm" (at 215 180 0) (effects (font (size 0.9 0.9)) (hide yes)))
+		(property "Datasheet" "~" (at 215 180 0) (effects (font (size 0.9 0.9)) (hide yes)))
+		(property "Description" "ENKU R0.1 bring-up test point" (at 215 180 0) (effects (font (size 0.9 0.9)) (hide yes)))
+		(pin "1")
+		(instances (project "enku-mainboard-r0.1" (path "/10000000-0000-4000-8000-000000000001/10000000-0000-4000-8000-000000000010" (reference "TP_SYS_EN") (unit 1))))
+	)
+	(global_label "SYS_EN" (shape bidirectional) (at 211.19 180 0)
+		(effects (font (size 0.9 0.9)) (justify right bottom))
+)
+	(symbol (lib_id "ENKU:TESTPOINT") (at 245 180 0) (unit 1) (exclude_from_sim no) (in_bom yes) (on_board yes) (dnp no)
+		(property "Reference" "TP_REG_PG" (at 245 177.46 0) (effects (font (size 0.9 0.9))))
+		(property "Value" "REG_PG" (at 245 182.54 0) (effects (font (size 0.9 0.9))))
+		(property "Footprint" "TestPoint:TestPoint_Pad_D1.5mm" (at 245 180 0) (effects (font (size 0.9 0.9)) (hide yes)))
+		(property "Datasheet" "~" (at 245 180 0) (effects (font (size 0.9 0.9)) (hide yes)))
+		(property "Description" "ENKU R0.1 bring-up test point" (at 245 180 0) (effects (font (size 0.9 0.9)) (hide yes)))
+		(pin "1")
+		(instances (project "enku-mainboard-r0.1" (path "/10000000-0000-4000-8000-000000000001/10000000-0000-4000-8000-000000000010" (reference "TP_REG_PG") (unit 1))))
+	)
+	(global_label "REG_PG" (shape bidirectional) (at 241.19 180 0)
+		(effects (font (size 0.9 0.9)) (justify right bottom))
+)
 	(sheet_instances (path "/" (page "2")))
 )

Commit message: Bind power ICs to local verified footprints
Parts:
- U_SRC: footprint ENKU:TPS2121_RUX0012B -> ENKU:TPS2121_RUX0012A
Changed lines of the file:
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@@
 		(property "Reference" "U_SRC" (at 48 46 0) (effects (font (size 0.95 0.95))))
 		(property "Value" "TPS2121" (at 76 46 0) (effects (font (size 0.95 0.95))))
-		(property "Footprint" "ENKU:TPS2121_RUX0012B" (at 62 62 0) (effects (font (size 0.95 0.95)) (hide yes)))
+		(property "Footprint" "ENKU:TPS2121_RUX0012A" (at 62 62 0) (effects (font (size 0.95 0.95)) (hide yes)))
 		(property "Datasheet" "~" (at 62 62 0) (effects (font (size 0.95 0.95)) (hide yes)))
 		(property "Description" "TPS2121" (at 62 62 0) (effects (font (size 0.95 0.95)) (hide yes)))
