File: hardware/kicad/enku-mainboard-r0.1/power.kicad_sch (KiCad schematic)
At the start: 42 parts

Commit message: schematic: normalize power reference designators
Parts:
- renumbered C_MUX_SS to C1, C_3V3_IN_HF to C10, C_3V3_OUT1 to C11, C_3V3_OUT2 to C12, C_USB_IN to C2, C_DOCK_IN to C3, C_MUX_OUT to C4, C_CHG_IN to C5, C_CHG_IN_HF to C6, C_CHG_SYS to C7, C_CHG_BAT to C8, C_3V3_IN to C9, J_BAT to J1, L_3V3 to L1, R_MUX_ILIM to R1, R_CHG_CE_PD to R10, R_STAT1_PU to R11, R_STAT2_PU to R12, R_SYS_EN_PD to R13, R_3V3_FB_TOP to R14, R_3V3_FB_BOT to R15, R_3V3_PG_PU to R16, R_PR1_USB to R2, R_PR1_GND to R3, R_CP2_DOCK to R4, R_CP2_GND to R5, R_OV1_GND to R6, R_OV2_GND to R7, R_CHG_ILIM_VSET to R8, R_CHG_ISET to R9, SW_POWER to SW1, TP_GND_PWR to TP1, TP_VBUS_USB to TP2, TP_VBUS_DOCK to TP3, TP_VBAT to TP4, TP_VSYS to TP5, TP_3V3 to TP6, TP_SYS_EN to TP7, TP_REG_PG to TP8, U_SRC to U2, U_CHG to U3, U_3V3 to U4

Commit message: schematic: align battery and hard-power footprints with PCB
Parts:
- J1: footprint Connector_Generic:Conn_01x03 -> Connector_Generic:JST_PH_3_PLACEMENT
- SW1: footprint Button_Switch_SMD:SW_SPST -> ENKU:HARD_POWER_SWITCH_PLACEMENT
Changed lines of the file:
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@@
 		(property "Reference" "J1" (at 128.255 109.73 0) (effects (font (size 0.95 0.95))))
 		(property "Value" "1S LiPo + NTC" (at 142.255 109.73 0) (effects (font (size 0.95 0.95))))
-		(property "Footprint" "Connector_Generic:Conn_01x03" (at 135.255 125.73 0) (effects (font (size 0.95 0.95)) (hide yes)))
+		(property "Footprint" Connector_Generic:JST_PH_3_PLACEMENT"Connector_Generic:Conn_01x03" (at 135.255 125.73 0) (effects (font (size 0.95 0.95)) (hide yes)))
 		(property "Datasheet" "~" (at 135.255 125.73 0) (effects (font (size 0.95 0.95)) (hide yes)))
 		(property "Description" "1S LiPo + NTC" (at 135.255 125.73 0) (effects (font (size 0.95 0.95)) (hide yes)))
@@
 		(property "Reference" "SW1" (at 199.105 111 0) (effects (font (size 0.95 0.95))))
 		(property "Value" "HARD POWER" (at 211.105 111 0) (effects (font (size 0.95 0.95))))
-		(property "Footprint" "Button_Switch_SMD:SW_SPST" (at 205.105 127 0) (effects (font (size 0.95 0.95)) (hide yes)))
+		(property "Footprint" ENKU:HARD_POWER_SWITCH_PLACEMENT"Button_Switch_SMD:SW_SPST" (at 205.105 127 0) (effects (font (size 0.95 0.95)) (hide yes)))
 		(property "Datasheet" "~" (at 205.105 127 0) (effects (font (size 0.95 0.95)) (hide yes)))
 		(property "Description" "HARD POWER" (at 205.105 127 0) (effects (font (size 0.95 0.95)) (hide yes)))
