File: hardware/kicad/enku-mainboard-r0.1/epd_hv.kicad_sch (KiCad schematic)
At the start: 27 parts

Commit message: Add R0.1 EPD HV measurement test points
Parts:
- added TP_EPD_GDR: EPD_GDR, TestPoint:TestPoint_Pad_D1.5mm, symbol ENKU:TESTPOINT
- added TP_EPD_RESE: EPD_RESE, TestPoint:TestPoint_Pad_D1.5mm, symbol ENKU:TESTPOINT
- added TP_EPD_VCOM: EPD_VCOM, TestPoint:TestPoint_Pad_D1.5mm, symbol ENKU:TESTPOINT
- added TP_EPD_VGH: EPD_VGH, TestPoint:TestPoint_Pad_D1.5mm, symbol ENKU:TESTPOINT
- added TP_EPD_VGL: EPD_VGL, TestPoint:TestPoint_Pad_D1.5mm, symbol ENKU:TESTPOINT
- added TP_GND_EPD: GND, TestPoint:TestPoint_Pad_D1.5mm, symbol ENKU:TESTPOINT
Connections:
- net EPD_GDR: now also TP_EPD_GDR.1 (TP)
- net EPD_RESE: now also TP_EPD_RESE.1 (TP)
- net EPD_VCOM: now also TP_EPD_VCOM.1 (TP)
- net EPD_VGH: now also TP_EPD_VGH.1 (TP)
- net EPD_VGL: now also TP_EPD_VGL.1 (TP)
- net GND: now also TP_GND_EPD.1 (TP)
Changed lines of the file:
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@@
 	(text "VPP is explicitly left NC for normal operation; BS1 is tied LOW for 4-wire SPI. Current panel pins 6/7 remain NC pending panel-specific continuity confirmation." (exclude_from_sim no) (at 25 30 0) (effects (font (size 1.0 1.0)) (justify left bottom)))
 	(text "R0.1 requires first-board scope validation of VGH/VGL/VSH/VSL/VCOM. TYS5040100M-10 and TYS5040470M-10 share the same TYS5040 land pattern, so 47uH remains a laboratory alternate without PCB respin." (exclude_from_sim no) (at 25 35 0) (effects (font (size 1.0 1.0)) (justify left bottom)))
+	(symbol (lib_id "ENKU:TESTPOINT") (at 45 200 0) (unit 1) (exclude_from_sim no) (in_bom yes) (on_board yes) (dnp no)
+		(property "Reference" "TP_EPD_GDR" (at 45 197.46 0) (effects (font (size 0.9 0.9))))
+		(property "Value" "EPD_GDR" (at 45 202.54 0) (effects (font (size 0.9 0.9))))
+		(property "Footprint" "TestPoint:TestPoint_Pad_D1.5mm" (at 45 200 0) (effects (font (size 0.9 0.9)) (hide yes)))
+		(property "Datasheet" "~" (at 45 200 0) (effects (font (size 0.9 0.9)) (hide yes)))
+		(property "Description" "ENKU R0.1 bring-up test point" (at 45 200 0) (effects (font (size 0.9 0.9)) (hide yes)))
+		(pin "1")
+		(instances (project "enku-mainboard-r0.1" (path "/10000000-0000-4000-8000-000000000001/10000000-0000-4000-8000-000000000030" (reference "TP_EPD_GDR") (unit 1))))
+	)
+	(global_label "EPD_GDR" (shape bidirectional) (at 41.19 200 0)
+		(effects (font (size 0.9 0.9)) (justify right bottom))
+)
+	(symbol (lib_id "ENKU:TESTPOINT") (at 80 200 0) (unit 1) (exclude_from_sim no) (in_bom yes) (on_board yes) (dnp no)
+		(property "Reference" "TP_EPD_RESE" (at 80 197.46 0) (effects (font (size 0.9 0.9))))
+		(property "Value" "EPD_RESE" (at 80 202.54 0) (effects (font (size 0.9 0.9))))
+		(property "Footprint" "TestPoint:TestPoint_Pad_D1.5mm" (at 80 200 0) (effects (font (size 0.9 0.9)) (hide yes)))
+		(property "Datasheet" "~" (at 80 200 0) (effects (font (size 0.9 0.9)) (hide yes)))
+		(property "Description" "ENKU R0.1 bring-up test point" (at 80 200 0) (effects (font (size 0.9 0.9)) (hide yes)))
+		(pin "1")
+		(instances (project "enku-mainboard-r0.1" (path "/10000000-0000-4000-8000-000000000001/10000000-0000-4000-8000-000000000030" (reference "TP_EPD_RESE") (unit 1))))
+	)
+	(global_label "EPD_RESE" (shape bidirectional) (at 76.19 200 0)
+		(effects (font (size 0.9 0.9)) (justify right bottom))
+)
+	(symbol (lib_id "ENKU:TESTPOINT") (at 115 200 0) (unit 1) (exclude_from_sim no) (in_bom yes) (on_board yes) (dnp no)
+		(property "Reference" "TP_EPD_VGH" (at 115 197.46 0) (effects (font (size 0.9 0.9))))
+		(property "Value" "EPD_VGH" (at 115 202.54 0) (effects (font (size 0.9 0.9))))
+		(property "Footprint" "TestPoint:TestPoint_Pad_D1.5mm" (at 115 200 0) (effects (font (size 0.9 0.9)) (hide yes)))
+		(property "Datasheet" "~" (at 115 200 0) (effects (font (size 0.9 0.9)) (hide yes)))
+		(property "Description" "ENKU R0.1 bring-up test point" (at 115 200 0) (effects (font (size 0.9 0.9)) (hide yes)))
+		(pin "1")
+		(instances (project "enku-mainboard-r0.1" (path "/10000000-0000-4000-8000-000000000001/10000000-0000-4000-8000-000000000030" (reference "TP_EPD_VGH") (unit 1))))
+	)
+	(global_label "EPD_VGH" (shape bidirectional) (at 111.19 200 0)
+		(effects (font (size 0.9 0.9)) (justify right bottom))
+)
+	(symbol (lib_id "ENKU:TESTPOINT") (at 150 200 0) (unit 1) (exclude_from_sim no) (in_bom yes) (on_board yes) (dnp no)
+		(property "Reference" "TP_EPD_VGL" (at 150 197.46 0) (effects (font (size 0.9 0.9))))
+		(property "Value" "EPD_VGL" (at 150 202.54 0) (effects (font (size 0.9 0.9))))
+		(property "Footprint" "TestPoint:TestPoint_Pad_D1.5mm" (at 150 200 0) (effects (font (size 0.9 0.9)) (hide yes)))
+		(property "Datasheet" "~" (at 150 200 0) (effects (font (size 0.9 0.9)) (hide yes)))
+		(property "Description" "ENKU R0.1 bring-up test point" (at 150 200 0) (effects (font (size 0.9 0.9)) (hide yes)))
+		(pin "1")
+		(instances (project "enku-mainboard-r0.1" (path "/10000000-0000-4000-8000-000000000001/10000000-0000-4000-8000-000000000030" (reference "TP_EPD_VGL") (unit 1))))
+	)
+	(global_label "EPD_VGL" (shape bidirectional) (at 146.19 200 0)
+		(effects (font (size 0.9 0.9)) (justify right bottom))
+)
+	(symbol (lib_id "ENKU:TESTPOINT") (at 185 200 0) (unit 1) (exclude_from_sim no) (in_bom yes) (on_board yes) (dnp no)
+		(property "Reference" "TP_EPD_VCOM" (at 185 197.46 0) (effects (font (size 0.9 0.9))))
+		(property "Value" "EPD_VCOM" (at 185 202.54 0) (effects (font (size 0.9 0.9))))
+		(property "Footprint" "TestPoint:TestPoint_Pad_D1.5mm" (at 185 200 0) (effects (font (size 0.9 0.9)) (hide yes)))
+		(property "Datasheet" "~" (at 185 200 0) (effects (font (size 0.9 0.9)) (hide yes)))
+		(property "Description" "ENKU R0.1 bring-up test point" (at 185 200 0) (effects (font (size 0.9 0.9)) (hide yes)))
+		(pin "1")
+		(instances (project "enku-mainboard-r0.1" (path "/10000000-0000-4000-8000-000000000001/10000000-0000-4000-8000-000000000030" (reference "TP_EPD_VCOM") (unit 1))))
+	)
+	(global_label "EPD_VCOM" (shape bidirectional) (at 181.19 200 0)
+		(effects (font (size 0.9 0.9)) (justify right bottom))
+)
+	(symbol (lib_id "ENKU:TESTPOINT") (at 220 200 0) (unit 1) (exclude_from_sim no) (in_bom yes) (on_board yes) (dnp no)
+		(property "Reference" "TP_GND_EPD" (at 220 197.46 0) (effects (font (size 0.9 0.9))))
+		(property "Value" "GND" (at 220 202.54 0) (effects (font (size 0.9 0.9))))
+		(property "Footprint" "TestPoint:TestPoint_Pad_D1.5mm" (at 220 200 0) (effects (font (size 0.9 0.9)) (hide yes)))
+		(property "Datasheet" "~" (at 220 200 0) (effects (font (size 0.9 0.9)) (hide yes)))
+		(property "Description" "ENKU R0.1 bring-up test point" (at 220 200 0) (effects (font (size 0.9 0.9)) (hide yes)))
+		(pin "1")
+		(instances (project "enku-mainboard-r0.1" (path "/10000000-0000-4000-8000-000000000001/10000000-0000-4000-8000-000000000030" (reference "TP_GND_EPD") (unit 1))))
+	)
+	(global_label "GND" (shape bidirectional) (at 216.19 200 0)
+		(effects (font (size 0.9 0.9)) (justify right bottom))
+)
 	(sheet_instances (path "/" (page "4")))
 )

Commit message: Bind EPD FPC to verified Hirose footprint
Parts:
- J_EPD: footprint ENKU:R0.1_FH34SRJ_24_DUAL_CONTACT_PLACEHOLDER -> ENKU:FH34SRJ-24S-0.5SH
Changed lines of the file:
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@@
 		(property "Reference" "J_EPD" (at 211 72 0) (effects (font (size 0.9 0.9))))
 		(property "Value" "FH34SRJ-24S-0.5SH(50)" (at 245 72 0) (effects (font (size 0.9 0.9))))
-		(property "Footprint" "ENKU:R0.1_FH34SRJ_24_DUAL_CONTACT_PLACEHOLDER" (at 228 86 0) (effects (font (size 0.9 0.9)) (hide yes)))
+		(property "Footprint" "ENKU:FH34SRJ-24S-0.5SH" (at 228 86 0) (effects (font (size 0.9 0.9)) (hide yes)))
 		(property "Datasheet" "~" (at 228 86 0) (effects (font (size 0.9 0.9)) (hide yes)))
 		(property "Description" "FH34SRJ-24S-0.5SH(50)" (at 228 86 0) (effects (font (size 0.9 0.9)) (hide yes)))
