File: hardware/kicad/enku-mainboard-r0.1/epd_hv.kicad_sch (KiCad schematic)
At the start: 33 parts

Commit message: Fix KiCad pin-label Y transform in epd_hv
Connections:
- net 3V3_SYS: now also J_EPD.15 (VDDIO); no longer J_EPD.22 (VSL)
- net EPD_BS1: now also J_EPD.8 (BS1); no longer J_EPD.5 (VSH2)
- net EPD_BUSY: now also J_EPD.9 (BUSY); no longer J_EPD.4 (NC)
- net EPD_CS_PANEL: now also J_EPD.12 (CS#); no longer J_EPD.1 (NC)
- net EPD_DC_PANEL: now also J_EPD.11 (D/C#); no longer J_EPD.2 (GDR)
- net EPD_GDR: now also J_EPD.2 (GDR), Q_EPD.1 (G); no longer J_EPD.11 (D/C#), Q_EPD.3 (D)
- net EPD_MOSI_PANEL: now also J_EPD.14 (SDA); no longer J_EPD.23 (VGL)
- net EPD_RESE: now also J_EPD.3 (RESE); no longer J_EPD.10 (RES#)
- net EPD_RST_PANEL: now also J_EPD.10 (RES#); no longer J_EPD.3 (RESE)
- net EPD_SCLK_PANEL: now also J_EPD.13 (SCL); no longer J_EPD.24 (VCOM)
- net EPD_SW: now also Q_EPD.3 (D); no longer Q_EPD.1 (G)
- net EPD_VCI: now also J_EPD.16 (VCI); no longer J_EPD.21 (VGH)
- net EPD_VCOM: now also J_EPD.24 (VCOM); no longer J_EPD.13 (SCL)
- net EPD_VDD: now also J_EPD.18 (VDD); no longer J_EPD.19 (VPP)
- net EPD_VGH: now also J_EPD.21 (VGH); no longer J_EPD.16 (VCI)
- net EPD_VGL: now also J_EPD.23 (VGL); no longer J_EPD.14 (SDA)
- net EPD_VSH1: now also J_EPD.20 (VSH1); no longer J_EPD.17 (VSS)
- net EPD_VSH2: now also J_EPD.5 (VSH2); no longer J_EPD.8 (BS1)
- net EPD_VSL: now also J_EPD.22 (VSL); no longer J_EPD.15 (VDDIO)
- net GND: now also J_EPD.17 (VSS), J_EPD.S1 (SHIELD), J_EPD.S2 (SHIELD); no longer J_EPD.20 (VSH1)
Changed lines of the file:
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@@
 		(instances (project "enku-mainboard-r0.1" (path "/10000000-0000-4000-8000-000000000001/10000000-0000-4000-8000-000000000030" (reference "J_EPD") (unit 1))))
 	)
-	(global_label "EPD_GDR" (shape input) (at 208.46 97.42999999999999 0) (effects (font (size 0.9 0.9)) (justify right bottom)))
-	(global_label "EPD_RESE" (shape input) (at 208.46 94.89 0) (effects (font (size 0.9 0.9)) (justify right bottom)))
-	(global_label "EPD_VSH2" (shape input) (at 208.46 89.81 0) (effects (font (size 0.9 0.9)) (justify right bottom)))
-	(global_label "EPD_BS1" (shape input) (at 208.46 82.19 0) (effects (font (size 0.9 0.9)) (justify right bottom)))
-	(global_label "EPD_BUSY" (shape input) (at 208.46 79.65 0) (effects (font (size 0.9 0.9)) (justify right bottom)))
-	(global_label "EPD_RST_PANEL" (shape input) (at 208.46 77.11 0) (effects (font (size 0.9 0.9)) (justify right bottom)))
-	(global_label "EPD_DC_PANEL" (shape input) (at 208.46 74.57 0) (effects (font (size 0.9 0.9)) (justify right bottom)))
-	(global_label "EPD_CS_PANEL" (shape input) (at 208.46 72.03 0) (effects (font (size 0.9 0.9)) (justify right bottom)))
-	(global_label "EPD_SCLK_PANEL" (shape output) (at 247.54 99.97 180) (effects (font (size 0.9 0.9)) (justify right bottom)))
-	(global_label "EPD_MOSI_PANEL" (shape output) (at 247.54 97.42999999999999 180) (effects (font (size 0.9 0.9)) (justify right bottom)))
-	(global_label "3V3_SYS" (shape output) (at 247.54 94.89 180) (effects (font (size 0.9 0.9)) (justify right bottom)))
-	(global_label "EPD_VCI" (shape output) (at 247.54 92.35 180) (effects (font (size 0.9 0.9)) (justify right bottom)))
-	(global_label "GND" (shape output) (at 247.54 89.81 180) (effects (font (size 0.9 0.9)) (justify right bottom)))
-	(global_label "EPD_VDD" (shape output) (at 247.54 87.27 180) (effects (font (size 0.9 0.9)) (justify right bottom)))
-	(global_label "EPD_VSH1" (shape output) (at 247.54 82.19 180) (effects (font (size 0.9 0.9)) (justify right bottom)))
-	(global_label "EPD_VGH" (shape output) (at 247.54 79.65 180) (effects (font (size 0.9 0.9)) (justify right bottom)))
-	(global_label "EPD_VSL" (shape output) (at 247.54 77.11 180) (effects (font (size 0.9 0.9)) (justify right bottom)))
-	(global_label "EPD_VGL" (shape output) (at 247.54 74.57 180) (effects (font (size 0.9 0.9)) (justify right bottom)))
-	(global_label "EPD_VCOM" (shape output) (at 247.54 72.03 180) (effects (font (size 0.9 0.9)) (justify right bottom)))
-	(no_connect (at 208.46 99.97))
-	(no_connect (at 208.46 92.35))
+	(global_label "EPD_GDR" (shape input) (at 208.46 74.57 0) (effects (font (size 0.9 0.9)) (justify right bottom)))
+	(global_label "EPD_RESE" (shape input) (at 208.46 77.11 0) (effects (font (size 0.9 0.9)) (justify right bottom)))
+	(global_label "EPD_VSH2" (shape input) (at 208.46 82.19 0) (effects (font (size 0.9 0.9)) (justify right bottom)))
+	(global_label "EPD_BS1" (shape input) (at 208.46 89.81 0) (effects (font (size 0.9 0.9)) (justify right bottom)))
+	(global_label "EPD_BUSY" (shape input) (at 208.46 92.35 0) (effects (font (size 0.9 0.9)) (justify right bottom)))
+	(global_label "EPD_RST_PANEL" (shape input) (at 208.46 94.89 0) (effects (font (size 0.9 0.9)) (justify right bottom)))
+	(global_label "EPD_DC_PANEL" (shape input) (at 208.46 97.43 0) (effects (font (size 0.9 0.9)) (justify right bottom)))
+	(global_label "EPD_CS_PANEL" (shape input) (at 208.46 99.97 0) (effects (font (size 0.9 0.9)) (justify right bottom)))
+	(global_label "EPD_SCLK_PANEL" (shape output) (at 247.54 72.03 180) (effects (font (size 0.9 0.9)) (justify right bottom)))
+	(global_label "EPD_MOSI_PANEL" (shape output) (at 247.54 74.57 180) (effects (font (size 0.9 0.9)) (justify right bottom)))
+	(global_label "3V3_SYS" (shape output) (at 247.54 77.11 180) (effects (font (size 0.9 0.9)) (justify right bottom)))
+	(global_label "EPD_VCI" (shape output) (at 247.54 79.65 180) (effects (font (size 0.9 0.9)) (justify right bottom)))
+	(global_label "GND" (shape output) (at 247.54 82.19 180) (effects (font (size 0.9 0.9)) (justify right bottom)))
+	(global_label "EPD_VDD" (shape output) (at 247.54 84.73 180) (effects (font (size 0.9 0.9)) (justify right bottom)))
+	(global_label "EPD_VSH1" (shape output) (at 247.54 89.81 180) (effects (font (size 0.9 0.9)) (justify right bottom)))
+	(global_label "EPD_VGH" (shape output) (at 247.54 92.35 180) (effects (font (size 0.9 0.9)) (justify right bottom)))
+	(global_label "EPD_VSL" (shape output) (at 247.54 94.89 180) (effects (font (size 0.9 0.9)) (justify right bottom)))
+	(global_label "EPD_VGL" (shape output) (at 247.54 97.43 180) (effects (font (size 0.9 0.9)) (justify right bottom)))
+	(global_label "EPD_VCOM" (shape output) (at 247.54 99.97 180) (effects (font (size 0.9 0.9)) (justify right bottom)))
+	(no_connect (at 208.46 72.03))
+	(no_connect (at 208.46 79.65))
+	(no_connect (at 208.46 84.73))
 	(no_connect (at 208.46 87.27))
-	(no_connect (at 208.46 84.73))
-	(no_connect (at 247.54 84.73))
+	(no_connect (at 247.54 87.27))
 	(symbol (lib_id "ENKU:R") (at 190 45 0) (unit 1) (exclude_from_sim no) (in_bom yes) (on_board yes) (dnp no)
 		(property "Reference" "R_EPD_VCI_LINK" (at 185 31 0) (effects (font (size 0.9 0.9))))
@@
 		(instances (project "enku-mainboard-r0.1" (path "/10000000-0000-4000-8000-000000000001/10000000-0000-4000-8000-000000000030" (reference "Q_EPD") (unit 1))))
 	)
-	(global_label "EPD_GDR" (shape input) (at 75.46000000000001 83.27 0) (effects (font (size 0.9 0.9)) (justify right bottom)))
+	(global_label "EPD_GDR" (shape input) (at 75.46 80.73 0) (effects (font (size 0.9 0.9)) (justify right bottom)))
 	(global_label "EPD_RESE" (shape output) (at 94.53999999999999 82 180) (effects (font (size 0.9 0.9)) (justify right bottom)))
-	(global_label "EPD_SW" (shape input) (at 75.46000000000001 80.72999999999999 0) (effects (font (size 0.9 0.9)) (justify right bottom)))
+	(global_label "EPD_SW" (shape input) (at 75.46 83.27 0) (effects (font (size 0.9 0.9)) (justify right bottom)))
 	(symbol (lib_id "ENKU:R") (at 85 108 0) (unit 1) (exclude_from_sim no) (in_bom yes) (on_board yes) (dnp no)
 		(property "Reference" "R_RESE" (at 80 94 0) (effects (font (size 0.9 0.9))))
@@
 	(global_label "EPD_VCI" (shape input) (at 47.46 118 0) (effects (font (size 0.9 0.9)) (justify right bottom)))
 	(global_label "GND" (shape output) (at 62.54 118 180) (effects (font (size 0.9 0.9)) (justify right bottom)))
-	(global_label "GND" (shape input) (at 208.46 69.49 0) (effects (font (size 0.9 0.9)) (justify right bottom)))
-	(global_label "GND" (shape input) (at 247.54 69.49 180) (effects (font (size 0.9 0.9)) (justify right bottom)))
+	(global_label "GND" (shape input) (at 208.46 102.51 0) (effects (font (size 0.9 0.9)) (justify right bottom)))
+	(global_label "GND" (shape input) (at 247.54 102.51 180) (effects (font (size 0.9 0.9)) (justify right bottom)))
 	(text "SSD1677 application circuit captured as discretes. R0.1 now follows the current 3.97-inch panel reference: 10uH + NMOS + 3x MBR0530 + 2.2R RESE + 1M GDR pulldown + local 4.7uF input capacitor." (exclude_from_sim no) (at 25 20 0) (effects (font (size 1.0 1.0)) (justify left bottom)))
 	(text "D1: SW -> VGH. C3 flying capacitor + D2/D3 form the negative VGL pump. Q_EPD source is sensed at RESE through 2.2R to GND." (exclude_from_sim no) (at 25 25 0) (effects (font (size 1.0 1.0)) (justify left bottom)))
