File: hardware/kicad/enku-mainboard-r0.1/epd_hv.kicad_sch (KiCad schematic)
At the start: 33 parts

Commit message: schematic: normalize epd_hv reference designators
Parts:
- renumbered C0_EPD_VCI to C22, C1_EPD_VDD to C23, C2_EPD_VGH to C24, C3_EPD_FLY to C25, C4_EPD_VGL to C26, C5_EPD_VSH1 to C27, C6_EPD_VSH2 to C28, C7_EPD_VSL to C29, C8_EPD_VCOM to C30, C_EPD_IN to C31, D1_EPD to D1, D2_EPD to D2, D3_EPD to D3, J_EPD to J3, L_EPD to L2, Q_EPD to Q1, R_EPD_VCI_LINK to R28, R_EPD_BS1 to R29, R_EPD_RST to R30, R_EPD_DC to R31, R_EPD_CS to R32, R_EPD_SCLK to R33, R_EPD_MOSI to R34, R_EPD_CS_PU to R35, R_EPD_RST_PU to R36, R_RESE to R37, R_GDR_PD to R38, TP_EPD_RESE to TP10, TP_EPD_VGH to TP11, TP_EPD_VGL to TP12, TP_EPD_VCOM to TP13, TP_GND_EPD to TP14, TP_EPD_GDR to TP9
