File: hardware/kicad/enku-mainboard-r0.1/frontlight.kicad_sch (KiCad schematic)
At the start: 33 parts

Commit message: Fix KiCad pin-label Y transform in frontlight
Connections:
- net FL_COOL_PWM: now also Q_FL_COOL.1 (G); no longer Q_FL_COOL.3 (D)
- net FL_COOL_RETURN: now also Q_FL_COOL.3 (D); no longer Q_FL_COOL.1 (G)
- net FL_FB: now also U_FL.3 (FB); no longer U_FL.1 (VIN)
- net FL_RAW1: now also J_FL.1 (RAW1); no longer J_FL.3 (RAW3)
- net FL_RAW3: now also J_FL.3 (RAW3); no longer J_FL.1 (RAW1)
- net FL_RAW4: now also J_FL.4 (RAW4); no longer J_FL.6 (RAW6)
- net FL_RAW6: now also J_FL.6 (RAW6); no longer J_FL.4 (RAW4)
- net FL_SW: now also U_FL.6 (SW); no longer U_FL.4 (GND)
- net FL_WARM_PWM: now also Q_FL_WARM.1 (G); no longer Q_FL_WARM.3 (D)
- net FL_WARM_RETURN: now also Q_FL_WARM.3 (D); no longer Q_FL_WARM.1 (G)
- net GND: now also J_FL.S1 (SHIELD), J_FL.S2 (SHIELD), U_FL.4 (GND); no longer U_FL.6 (SW)
- net VSYS: now also U_FL.1 (VIN); no longer U_FL.3 (FB)
Changed lines of the file:
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@@
 		(instances (project "enku-mainboard-r0.1" (path "/10000000-0000-4000-8000-000000000001/10000000-0000-4000-8000-000000000040" (reference "U_FL") (unit 1))))
 	)
-	(global_label "VSYS" (shape input) (at 56.46 67.54 0) (effects (font (size 0.9 0.9)) (justify right bottom)))
+	(global_label "VSYS" (shape input) (at 56.46 62.46 0) (effects (font (size 0.9 0.9)) (justify right bottom)))
 	(global_label "FL_ADIM" (shape input) (at 56.46 65 0) (effects (font (size 0.9 0.9)) (justify right bottom)))
-	(global_label "FL_FB" (shape input) (at 56.46 62.46000000000001 0) (effects (font (size 0.9 0.9)) (justify right bottom)))
-	(global_label "GND" (shape output) (at 83.53999999999999 62.46000000000001 180) (effects (font (size 0.9 0.9)) (justify right bottom)))
+	(global_label "FL_FB" (shape input) (at 56.46 67.54 0) (effects (font (size 0.9 0.9)) (justify right bottom)))
+	(global_label "GND" (shape output) (at 83.54 67.54 180) (effects (font (size 0.9 0.9)) (justify right bottom)))
 	(global_label "FL_LED_PLUS" (shape output) (at 83.53999999999999 65 180) (effects (font (size 0.9 0.9)) (justify right bottom)))
-	(global_label "FL_SW" (shape output) (at 83.53999999999999 67.54 180) (effects (font (size 0.9 0.9)) (justify right bottom)))
+	(global_label "FL_SW" (shape output) (at 83.54 62.46 180) (effects (font (size 0.9 0.9)) (justify right bottom)))
 	(symbol (lib_id "ENKU:L") (at 35 65 0) (unit 1) (exclude_from_sim no) (in_bom yes) (on_board yes) (dnp no)
 		(property "Reference" "L_FL" (at 30 51 0) (effects (font (size 0.9 0.9))))
@@
 		(instances (project "enku-mainboard-r0.1" (path "/10000000-0000-4000-8000-000000000001/10000000-0000-4000-8000-000000000040" (reference "Q_FL_WARM") (unit 1))))
 	)
-	(global_label "FL_WARM_PWM" (shape input) (at 115.46000000000001 63.27 0) (effects (font (size 0.9 0.9)) (justify right bottom)))
+	(global_label "FL_WARM_PWM" (shape input) (at 115.46 60.73 0) (effects (font (size 0.9 0.9)) (justify right bottom)))
 	(global_label "FL_FB" (shape output) (at 134.54 62 180) (effects (font (size 0.9 0.9)) (justify right bottom)))
-	(global_label "FL_WARM_RETURN" (shape input) (at 115.46000000000001 60.730000000000004 0) (effects (font (size 0.9 0.9)) (justify right bottom)))
+	(global_label "FL_WARM_RETURN" (shape input) (at 115.46 63.27 0) (effects (font (size 0.9 0.9)) (justify right bottom)))
 	(symbol (lib_id "ENKU:BSS138") (at 125 92 0) (unit 1) (exclude_from_sim no) (in_bom yes) (on_board yes) (dnp no)
 		(property "Reference" "Q_FL_COOL" (at 118 78 0) (effects (font (size 0.9 0.9))))
@@
 		(instances (project "enku-mainboard-r0.1" (path "/10000000-0000-4000-8000-000000000001/10000000-0000-4000-8000-000000000040" (reference "Q_FL_COOL") (unit 1))))
 	)
-	(global_label "FL_COOL_PWM" (shape input) (at 115.46000000000001 93.27 0) (effects (font (size 0.9 0.9)) (justify right bottom)))
+	(global_label "FL_COOL_PWM" (shape input) (at 115.46 90.73 0) (effects (font (size 0.9 0.9)) (justify right bottom)))
 	(global_label "FL_FB" (shape output) (at 134.54 92 180) (effects (font (size 0.9 0.9)) (justify right bottom)))
-	(global_label "FL_COOL_RETURN" (shape input) (at 115.46000000000001 90.72999999999999 0) (effects (font (size 0.9 0.9)) (justify right bottom)))
+	(global_label "FL_COOL_RETURN" (shape input) (at 115.46 93.27 0) (effects (font (size 0.9 0.9)) (justify right bottom)))
 	(symbol (lib_id "ENKU:R") (at 150 62 0) (unit 1) (exclude_from_sim no) (in_bom yes) (on_board yes) (dnp no)
 		(property "Reference" "R_FL_WARM_PD" (at 145 48 0) (effects (font (size 0.9 0.9))))
@@
 		(instances (project "enku-mainboard-r0.1" (path "/10000000-0000-4000-8000-000000000001/10000000-0000-4000-8000-000000000040" (reference "J_FL") (unit 1))))
 	)
-	(global_label "FL_RAW1" (shape input) (at 213.46 84.54 0) (effects (font (size 0.9 0.9)) (justify right bottom)))
+	(global_label "FL_RAW1" (shape input) (at 213.46 79.46 0) (effects (font (size 0.9 0.9)) (justify right bottom)))
 	(global_label "FL_RAW2" (shape input) (at 213.46 82 0) (effects (font (size 0.9 0.9)) (justify right bottom)))
-	(global_label "FL_RAW3" (shape input) (at 213.46 79.46000000000001 0) (effects (font (size 0.9 0.9)) (justify right bottom)))
-	(global_label "FL_RAW4" (shape output) (at 236.54 84.54 180) (effects (font (size 0.9 0.9)) (justify right bottom)))
+	(global_label "FL_RAW3" (shape input) (at 213.46 84.54 0) (effects (font (size 0.9 0.9)) (justify right bottom)))
+	(global_label "FL_RAW4" (shape output) (at 236.54 79.46 180) (effects (font (size 0.9 0.9)) (justify right bottom)))
 	(global_label "FL_RAW5" (shape output) (at 236.54 82 180) (effects (font (size 0.9 0.9)) (justify right bottom)))
-	(global_label "FL_RAW6" (shape output) (at 236.54 79.46000000000001 180) (effects (font (size 0.9 0.9)) (justify right bottom)))
+	(global_label "FL_RAW6" (shape output) (at 236.54 84.54 180) (effects (font (size 0.9 0.9)) (justify right bottom)))
 	(symbol (lib_id "ENKU:R") (at 175 42 0) (unit 1) (exclude_from_sim no) (in_bom yes) (on_board yes) (dnp yes)
 		(property "Reference" "R_FL_MAP1_P" (at 170 28 0) (effects (font (size 0.9 0.9))))
@@
 	(global_label "FL_RAW6" (shape input) (at 203.46 122 0) (effects (font (size 0.9 0.9)) (justify right bottom)))
 	(global_label "FL_COOL_RETURN" (shape output) (at 218.54 122 180) (effects (font (size 0.9 0.9)) (justify right bottom)))
-	(global_label "GND" (shape input) (at 213.46 76.92 0) (effects (font (size 0.9 0.9)) (justify right bottom)))
-	(global_label "GND" (shape input) (at 236.54 76.92 180) (effects (font (size 0.9 0.9)) (justify right bottom)))
+	(global_label "GND" (shape input) (at 213.46 87.08 0) (effects (font (size 0.9 0.9)) (justify right bottom)))
+	(global_label "GND" (shape input) (at 236.54 87.08 180) (effects (font (size 0.9 0.9)) (justify right bottom)))
 	(text "TPS923610 DRL pinout: VIN=1, ADIM=2, FB=3, GND=4, VOUT=5, SW=6. L_FL is between VSYS and SW; R_FL_SET is FB-to-GND." (exclude_from_sim no) (at 25 20 0) (effects (font (size 1.0 1.0)) (justify left bottom)))
 	(text "Warm/cool selectors switch each LED return into the common FB sense node. ADIM is the master brightness/shutdown input and has an explicit pulldown." (exclude_from_sim no) (at 25 25 0) (effects (font (size 1.0 1.0)) (justify left bottom)))
