File: hardware/kicad/enku-mainboard-r0.1/frontlight.kicad_sch (KiCad schematic)
At the start: 33 parts

Commit message: schematic: normalize frontlight reference designators
Parts:
- renumbered C_FL_IN to C32, C_FL_IN_HF to C33, C_FL_OUT to C34, J_FL to J4, L_FL to L3, Q_FL_WARM to Q2, Q_FL_COOL to Q3, R_FL_SET to R39, R_FL_ADIM_PD to R40, R_FL_ADIM_LINK to R41, R_FL_WARM_PD to R42, R_FL_COOL_PD to R43, R_FL_MAP1_P to R44, R_FL_MAP1_W to R45, R_FL_MAP1_C to R46, R_FL_MAP2_P to R47, R_FL_MAP2_W to R48, R_FL_MAP2_C to R49, R_FL_MAP3_P to R50, R_FL_MAP3_W to R51, R_FL_MAP3_C to R52, R_FL_MAP4_P to R53, R_FL_MAP4_W to R54, R_FL_MAP4_C to R55, R_FL_MAP5_P to R56, R_FL_MAP5_W to R57, R_FL_MAP5_C to R58, R_FL_MAP6_P to R59, R_FL_MAP6_W to R60, R_FL_MAP6_C to R61, TP_FL_LED_PLUS to TP15, TP_FL_FB to TP16, U_FL to U7
