File: hardware/kicad/enku-mainboard-r0.1/connectors.kicad_sch (KiCad schematic)
At the start: 15 parts

Commit message: schematic: normalize connectors reference designators
Parts:
- renumbered C_USB_SHIELD to C35, C_DOCK_DET to C36, J_USB to J5, J_DOCK to J6, J_DBG to J7, J_QI to J8, R_CC1 to R62, R_CC2 to R63, R_USB_DP to R64, R_USB_DM to R65, R_USB_SHIELD to R66, R_USB_SHIELD_0R to R67, R_DOCK_DET_SER to R68, R_DOCK_DET_PD to R69, U_USB_ESD to U8
