File: hardware/kicad/enku-mainboard-r0.1/mcu_io.kicad_sch (KiCad schematic)
At the start: 29 parts, among them U1 ESP32-S3-WROOM-1-N16R8

Commit message: schematic: normalize mcu_io reference designators
Parts:
- renumbered C_ESP_BULK to C13, C_ESP_HF to C14, C_EN to C15, C_SD_BULK to C16, C_SD_HF to C17, C_IMU_VDD to C18, C_IMU_VDDIO to C19, C_HALL to C20, C_BAT_ADC to C21, J_SD to J2, R_EN_PU to R17, R_BOOT_PU to R18, R_SD_CS to R19, R_SD_MOSI to R20, R_SD_SCLK to R21, R_SD_MISO to R22, R_SD_CS_PU to R23, R_I2C_SDA_PU to R24, R_I2C_SCL_PU to R25, R_BAT_TOP to R26, R_BAT_BOT to R27, SW_BOOT to SW2, SW_PREV to SW3, SW_NEXT to SW4, SW_SELECT to SW5, SW_BACK to SW6, U_IMU to U5, U_HALL to U6

Commit message: schematic: align intentional input footprints with PCB
Parts:
- SW3, SW4, SW5, SW6: footprint Button_Switch_SMD:SW_SPST_TL3342 -> ENKU:READING_BUTTON_PLACEMENT
Changed lines of the file:
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@@
 		(property "Reference" "SW3" (at 26.385 149.37 0) (effects (font (size 0.88 0.88))))
 		(property "Value" "BTN_PREV" (at 38.385 149.37 0) (effects (font (size 0.88 0.88))))
-		(property "Footprint" "Button_Switch_SMD:SW_SPST_TL3342" (at 32.385 166.37 0) (effects (font (size 0.88 0.88)) (hide yes)))
+		(property "Footprint" ENKU:READING_BUTTON_PLACEMENT"Button_Switch_SMD:SW_SPST_TL3342" (at 32.385 166.37 0) (effects (font (size 0.88 0.88)) (hide yes)))
 		(property "Datasheet" "~" (at 32.385 166.37 0) (effects (font (size 0.88 0.88)) (hide yes)))
 		(property "Description" "BTN_PREV" (at 32.385 166.37 0) (effects (font (size 0.88 0.88)) (hide yes)))
@@
 		(property "Reference" "SW4" (at 55.595 149.37 0) (effects (font (size 0.88 0.88))))
 		(property "Value" "BTN_NEXT" (at 67.595 149.37 0) (effects (font (size 0.88 0.88))))
-		(property "Footprint" "Button_Switch_SMD:SW_SPST_TL3342" (at 61.595 166.37 0) (effects (font (size 0.88 0.88)) (hide yes)))
+		(property "Footprint" ENKU:READING_BUTTON_PLACEMENT"Button_Switch_SMD:SW_SPST_TL3342" (at 61.595 166.37 0) (effects (font (size 0.88 0.88)) (hide yes)))
 		(property "Datasheet" "~" (at 61.595 166.37 0) (effects (font (size 0.88 0.88)) (hide yes)))
 		(property "Description" "BTN_NEXT" (at 61.595 166.37 0) (effects (font (size 0.88 0.88)) (hide yes)))
@@
 		(property "Reference" "SW5" (at 86.075 149.37 0) (effects (font (size 0.88 0.88))))
 		(property "Value" "BTN_SELECT" (at 98.075 149.37 0) (effects (font (size 0.88 0.88))))
-		(property "Footprint" "Button_Switch_SMD:SW_SPST_TL3342" (at 92.075 166.37 0) (effects (font (size 0.88 0.88)) (hide yes)))
+		(property "Footprint" ENKU:READING_BUTTON_PLACEMENT"Button_Switch_SMD:SW_SPST_TL3342" (at 92.075 166.37 0) (effects (font (size 0.88 0.88)) (hide yes)))
 		(property "Datasheet" "~" (at 92.075 166.37 0) (effects (font (size 0.88 0.88)) (hide yes)))
 		(property "Description" "BTN_SELECT" (at 92.075 166.37 0) (effects (font (size 0.88 0.88)) (hide yes)))
@@
 		(property "Reference" "SW6" (at 116.555 149.37 0) (effects (font (size 0.88 0.88))))
 		(property "Value" "BTN_BACK" (at 128.555 149.37 0) (effects (font (size 0.88 0.88))))
-		(property "Footprint" "Button_Switch_SMD:SW_SPST_TL3342" (at 122.555 166.37 0) (effects (font (size 0.88 0.88)) (hide yes)))
+		(property "Footprint" ENKU:READING_BUTTON_PLACEMENT"Button_Switch_SMD:SW_SPST_TL3342" (at 122.555 166.37 0) (effects (font (size 0.88 0.88)) (hide yes)))
 		(property "Datasheet" "~" (at 122.555 166.37 0) (effects (font (size 0.88 0.88)) (hide yes)))
 		(property "Description" "BTN_BACK" (at 122.555 166.37 0) (effects (font (size 0.88 0.88)) (hide yes)))
