File: hardware/kicad/enku-mainboard-r0.1/mcu_io.kicad_sch (KiCad schematic)
At the start: 29 parts, among them J2 Hirose DM3AT-SF-PEJM5, SW2 BOOT / RECOVERY, SW3 BTN_PREV, SW4 BTN_NEXT, SW5 BTN_SELECT, SW6 BTN_BACK, U1 ESP32-S3-WROOM-1-N16R8, U5 BMI270, U6 DRV5032FBDBZR

Commit message: schematic: bind locked ENKU microSD footprint
Parts:
- J2: footprint Connector_Card:microSD_HC_Hirose_DM3AT-SF-PEJM5 -> ENKU:MICROSD_DM3AT_ENKU
Changed lines of the file:
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@@
 		(property "Reference" "J2" (at 163.625 41.42 0) (effects (font (size 0.88 0.88))))
 		(property "Value" "Hirose DM3AT-SF-PEJM5" (at 185.625 41.42 0) (effects (font (size 0.88 0.88))))
-		(property "Footprint" "Connector_Card:microSD_HC_Hirose_DM3AT-SF-PEJM5" (at 174.625 58.42 0) (effects (font (size 0.88 0.88)) (hide yes)))
+		(property "Footprint" "ENKU:MICROSD_DM3AT_ENKU" (at 174.625 58.42 0) (effects (font (size 0.88 0.88)) (hide yes)))
 		(property "Datasheet" "~" (at 174.625 58.42 0) (effects (font (size 0.88 0.88)) (hide yes)))
 		(property "Description" "Hirose DM3AT-SF-PEJM5" (at 174.625 58.42 0) (effects (font (size 0.88 0.88)) (hide yes)))
