File: hardware/kicad/enku-mainboard-r0.1/enku-mainboard-r0.1.kicad_pcb (KiCad board)
At the start: 4 copper layers, 156 parts, among them J1 1S LiPo + NTC, J2 Hirose DM3AT-SF-PEJM5, J3 FH34SRJ-24S-0.5SH(50), J4 FH34SRJ-6S-0.5SH(50), J5 GCT USB4105-GF-A-120, J6 4-pin pogo dock, J7 Tag-Connect TC2030-IDC-NL, J8 Pro Wireless Qi raw interface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, Q1 IRLML6346TRPBF, Q2 BSS138LT1G, Q3 BSS138LT1G, SW1 HARD POWER, SW2 BOOT / RECOVERY, SW3 BTN_PREV, SW4 BTN_NEXT, SW5 BTN_SELECT, SW6 BTN_BACK, U1 ESP32-S3-WROOM-1-N16R8, U2 TPS2121, U3 BQ25185DLHR, U4 TPS63802DLAR, U5 BMI270, U6 DRV5032FBDBZR, U7 TPS923610DRLR, U8 USBLC6-2SC6

Commit message: pcb: rotate enable pulldown into clear right-side channel
Parts:
- moved R13 2.83 mm to (66.5, 96.5), turned to 90 degrees
Changed lines of the file:
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@@
     )
   (footprint "Resistor_SMD:R_0603_1608Metric" (layer "F.Cu")
-    (at 64.5 98.5 0)
+    (at 66.5 96.5 90)
       (property "Reference" "R13" (at 0 -1.45 0) (layer "F.SilkS") hide)
       (property "Value" "100k" (at 0 1.45 0) (layer "F.Fab") hide)
@@
   (segment (start 58.15 96.80) (end 58.15 94.40) (width 0.30) (layer "F.Cu") (net 2))
   (segment (start 57.10 90.00) (end 57.70 90.60) (width 0.18) (layer "F.Cu") (net 74))
-  (segment (start 57.70 90.60) (end 57.70 98.50) (width 0.18) (layer "F.Cu") (net 74))
-  (segment (start 57.70 98.50) (end 63.70 98.50) (width 0.18) (layer "F.Cu") (net 74))
+  (segment (start 57.70 90.60) (end 57.70 96.50) (width 0.18) (layer "F.Cu") (net 74))
+  (segment (start 57.70 96.50) (end 65.70 96.50) (width 0.18) (layer "F.Cu") (net 74))
   (segment (start 57.10 91.50) (end 56.45 91.50) (width 0.18) (layer "F.Cu") (net 77))
   (segment (start 56.45 91.50) (end 56.45 87.50) (width 0.18) (layer "F.Cu") (net 77))
