File: hardware/kicad/enku-mainboard-r0.1/enku-mainboard-r0.1.kicad_pcb (KiCad board)
At the start: 4 copper layers, 156 parts, among them J1 1S LiPo + NTC, J2 Hirose DM3AT-SF-PEJM5, J3 FH34SRJ-24S-0.5SH(50), J4 FH34SRJ-6S-0.5SH(50), J5 GCT USB4105-GF-A-120, J6 4-pin pogo dock, J7 Tag-Connect TC2030-IDC-NL, J8 Pro Wireless Qi raw interface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, Q1 IRLML6346TRPBF, Q2 BSS138LT1G, Q3 BSS138LT1G, SW1 HARD POWER, SW2 BOOT / RECOVERY, SW3 BTN_PREV, SW4 BTN_NEXT, SW5 BTN_SELECT, SW6 BTN_BACK, U1 ESP32-S3-WROOM-1-N16R8, U2 TPS2121, U3 BQ25185DLHR, U4 TPS63802DLAR, U5 BMI270, U6 DRV5032FBDBZR, U7 TPS923610DRLR, U8 USBLC6-2SC6

Commit message: pcb: move SD upper vias beyond dock pads
Routing:
- net SD_MOSI_CARD: track 22.7 -> 29.0 mm
- net SD_CS_CARD: track 23.6 -> 29.5 mm
Changed lines of the file:
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@@
   (segment (start 34 24.675) (end 34 23.8) (width 0.12) (layer "F.Cu") (net 22))
   (via (at 34 23.8) (size 0.55) (drill 0.25) (layers "F.Cu" "In1.Cu") (net 22))
-  (segment (start 43.525 98.8) (end 43.2 97.4) (width 0.18) (layer "F.Cu") (net 9))
-  (via (at 43.2 97.4) (size 0.60) (drill 0.30) (layers "F.Cu" "In1.Cu") (net 9))
-  (segment (start 43.2 97.4) (end 25.0 98.0) (width 0.18) (layer "In1.Cu") (net 9))
+  (segment (start 43.525 98.8) (end 46.8 97.0) (width 0.18) (layer "F.Cu") (net 9))
+  (via (at 46.8 97.0) (size 0.60) (drill 0.30) (layers "F.Cu" "In1.Cu") (net 9))
+  (segment (start 46.8 97.0) (end 25.0 98.0) (width 0.18) (layer "In1.Cu") (net 9))
   (via (at 25.0 98.0) (size 0.60) (drill 0.30) (layers "F.Cu" "In1.Cu") (net 9))
   (segment (start 25.0 98.0) (end 21.175 99.025) (width 0.18) (layer "F.Cu") (net 9))
-  (segment (start 43.525 101.5) (end 43.0 100.8) (width 0.18) (layer "F.Cu") (net 10))
-  (via (at 43.0 100.8) (size 0.60) (drill 0.30) (layers "F.Cu" "In1.Cu") (net 10))
-  (segment (start 43.0 100.8) (end 25.0 100.6) (width 0.18) (layer "In1.Cu") (net 10))
+  (segment (start 43.525 101.5) (end 46.8 100.8) (width 0.18) (layer "F.Cu") (net 10))
+  (via (at 46.8 100.8) (size 0.60) (drill 0.30) (layers "F.Cu" "In1.Cu") (net 10))
+  (segment (start 46.8 100.8) (end 25.0 100.6) (width 0.18) (layer "In1.Cu") (net 10))
   (via (at 25.0 100.6) (size 0.60) (drill 0.30) (layers "F.Cu" "In1.Cu") (net 10))
   (segment (start 25.0 100.6) (end 21.175 100.125) (width 0.18) (layer "F.Cu") (net 10))

Commit message: pcb: clear final SD card bundle short
Routing:
- net SD_CS_CARD: track 29.5 -> 30.2 mm
Changed lines of the file:
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@@
   (segment (start 34 24.675) (end 34 23.8) (width 0.12) (layer "F.Cu") (net 22))
   (via (at 34 23.8) (size 0.55) (drill 0.25) (layers "F.Cu" "In1.Cu") (net 22))
-  (segment (start 43.525 98.8) (end 46.8 97.0) (width 0.18) (layer "F.Cu") (net 9))
-  (via (at 46.8 97.0) (size 0.60) (drill 0.30) (layers "F.Cu" "In1.Cu") (net 9))
-  (segment (start 46.8 97.0) (end 25.0 98.0) (width 0.18) (layer "In1.Cu") (net 9))
+  (segment (start 43.525 98.8) (end 46.8 96.0) (width 0.18) (layer "F.Cu") (net 9))
+  (via (at 46.8 96.0) (size 0.60) (drill 0.30) (layers "F.Cu" "In1.Cu") (net 9))
+  (segment (start 46.8 96.0) (end 25.0 98.0) (width 0.18) (layer "In1.Cu") (net 9))
   (via (at 25.0 98.0) (size 0.60) (drill 0.30) (layers "F.Cu" "In1.Cu") (net 9))
   (segment (start 25.0 98.0) (end 21.175 99.025) (width 0.18) (layer "F.Cu") (net 9))

Commit message: pcb: dogleg SD CS around 3V3 via
Routing:
- net SD_CS_CARD: track 30.2 -> 34.5 mm
Changed lines of the file:
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@@
   (segment (start 43.525 98.8) (end 46.8 96.0) (width 0.18) (layer "F.Cu") (net 9))
   (via (at 46.8 96.0) (size 0.60) (drill 0.30) (layers "F.Cu" "In1.Cu") (net 9))
-  (segment (start 46.8 96.0) (end 25.0 98.0) (width 0.18) (layer "In1.Cu") (net 9))
+  (segment (start 46.8 96.0) (end 46.8 94.8) (width 0.18) (layer "In1.Cu") (net 9))
+  (segment (start 46.8 94.8) (end 25.0 94.8) (width 0.18) (layer "In1.Cu") (net 9))
+  (segment (start 25.0 94.8) (end 25.0 98.0) (width 0.18) (layer "In1.Cu") (net 9))
   (via (at 25.0 98.0) (size 0.60) (drill 0.30) (layers "F.Cu" "In1.Cu") (net 9))
   (segment (start 25.0 98.0) (end 21.175 99.025) (width 0.18) (layer "F.Cu") (net 9))

Commit message: pcb: close USB shield network
Routing:
- net CHG_STAT1: track 0.00 -> 31.2 mm, vias 0 -> 1
Changed lines of the file:
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@@
   (via (at 25.0 106.0) (size 0.60) (drill 0.30) (layers "F.Cu" "In1.Cu") (net 12))
   (segment (start 25.0 106.0) (end 21.175 104.525) (width 0.18) (layer "F.Cu") (net 12))
+  (segment (start 59.2 108.5) (end 62.2 108.5) (width 0.25) (layer "F.Cu") (net 52))
+  (segment (start 62.2 108.5) (end 65.2 108.5) (width 0.25) (layer "F.Cu") (net 52))
+  (segment (start 51.32 107.22) (end 51.32 111.4) (width 0.30) (layer "B.Cu") (net 52))
+  (segment (start 42.68 107.22) (end 42.68 111.4) (width 0.30) (layer "B.Cu") (net 52))
+  (segment (start 42.68 111.4) (end 51.32 111.4) (width 0.30) (layer "B.Cu") (net 52))
+  (segment (start 51.32 107.22) (end 57.0 107.22) (width 0.25) (layer "B.Cu") (net 52))
+  (via (at 57.0 107.22) (size 0.70) (drill 0.35) (layers "F.Cu" "B.Cu") (net 52))
+  (segment (start 57.0 107.22) (end 59.2 108.5) (width 0.25) (layer "F.Cu") (net 52))
 )
     (attr dnp)

Commit message: pcb: restore clean SD milestone after shield net mismatch
Routing:
- net CHG_STAT1: track 31.2 -> 0.00 mm, vias 1 -> 0
Changed lines of the file:
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@@
   (via (at 25.0 106.0) (size 0.60) (drill 0.30) (layers "F.Cu" "In1.Cu") (net 12))
   (segment (start 25.0 106.0) (end 21.175 104.525) (width 0.18) (layer "F.Cu") (net 12))
-  (segment (start 59.2 108.5) (end 62.2 108.5) (width 0.25) (layer "F.Cu") (net 52))
-  (segment (start 62.2 108.5) (end 65.2 108.5) (width 0.25) (layer "F.Cu") (net 52))
-  (segment (start 51.32 107.22) (end 51.32 111.4) (width 0.30) (layer "B.Cu") (net 52))
-  (segment (start 42.68 107.22) (end 42.68 111.4) (width 0.30) (layer "B.Cu") (net 52))
-  (segment (start 42.68 111.4) (end 51.32 111.4) (width 0.30) (layer "B.Cu") (net 52))
-  (segment (start 51.32 107.22) (end 57.0 107.22) (width 0.25) (layer "B.Cu") (net 52))
-  (via (at 57.0 107.22) (size 0.70) (drill 0.35) (layers "F.Cu" "B.Cu") (net 52))
-  (segment (start 57.0 107.22) (end 59.2 108.5) (width 0.25) (layer "F.Cu") (net 52))
 )
     (attr dnp)

Commit message: pcb: join USB shield network above conditioning row
Routing:
- net USB_SHIELD: track 0.00 -> 11.1 mm
Changed lines of the file:
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@@
   (via (at 25.0 106.0) (size 0.60) (drill 0.30) (layers "F.Cu" "In1.Cu") (net 12))
   (segment (start 25.0 106.0) (end 21.175 104.525) (width 0.18) (layer "F.Cu") (net 12))
+  (segment (start 59.2 108.5) (end 59.2 106.8) (width 0.20) (layer "F.Cu") (net 8))
+  (segment (start 59.2 106.8) (end 62.2 106.8) (width 0.20) (layer "F.Cu") (net 8))
+  (segment (start 62.2 106.8) (end 62.2 108.5) (width 0.20) (layer "F.Cu") (net 8))
+  (segment (start 62.2 106.8) (end 65.2 106.8) (width 0.20) (layer "F.Cu") (net 8))
+  (segment (start 65.2 106.8) (end 65.2 108.5) (width 0.20) (layer "F.Cu") (net 8))
 )
     (attr dnp)

Commit message: pcb: close USB ESD connector-side stubs
Routing:
- net USB_DP_CONN: track 19.7 -> 23.5 mm, vias 2 -> 3
- net USB_DM_CONN: track 10.3 -> 11.9 mm
Changed lines of the file:
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@@
   (segment (start 62.2 106.8) (end 65.2 106.8) (width 0.20) (layer "F.Cu") (net 8))
   (segment (start 65.2 106.8) (end 65.2 108.5) (width 0.20) (layer "F.Cu") (net 8))
+  (segment (start 55.3 107.85) (end 56.4 106.7) (width 0.15) (layer "F.Cu") (net 6))
+  (via (at 56.4 106.7) (size 0.55) (drill 0.25) (layers "F.Cu" "In1.Cu") (net 6))
+  (segment (start 56.4 106.7) (end 56.4 104.5) (width 0.15) (layer "In1.Cu") (net 6))
+  (segment (start 53.1 107.85) (end 52.55 108.4) (width 0.15) (layer "F.Cu") (net 7))
+  (segment (start 52.55 108.4) (end 52.55 109.2) (width 0.15) (layer "F.Cu") (net 7))
 )
     (attr dnp)

Commit message: pcb: connect USB connector pair to series resistors
Routing:
- net USB_DM_CONN: track 11.9 -> 27.3 mm, vias 0 -> 2
- net USB_DP_CONN: track 23.5 -> 28.5 mm, vias 3 -> 4
Changed lines of the file:
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@@
   (segment (start 53.1 107.85) (end 52.55 108.4) (width 0.15) (layer "F.Cu") (net 7))
   (segment (start 52.55 108.4) (end 52.55 109.2) (width 0.15) (layer "F.Cu") (net 7))
+  (segment (start 56.4 104.5) (end 58.0 103.0) (width 0.15) (layer "In1.Cu") (net 6))
+  (via (at 58.0 103.0) (size 0.55) (drill 0.25) (layers "F.Cu" "In1.Cu") (net 6))
+  (segment (start 58.0 103.0) (end 59.2 100.5) (width 0.15) (layer "F.Cu") (net 6))
+  (segment (start 52.55 109.2) (end 57.0 110.0) (width 0.15) (layer "F.Cu") (net 7))
+  (via (at 57.0 110.0) (size 0.55) (drill 0.25) (layers "F.Cu" "In1.Cu") (net 7))
+  (segment (start 57.0 110.0) (end 61.0 103.0) (width 0.15) (layer "In1.Cu") (net 7))
+  (via (at 61.0 103.0) (size 0.55) (drill 0.25) (layers "F.Cu" "In1.Cu") (net 7))
+  (segment (start 61.0 103.0) (end 62.2 100.5) (width 0.15) (layer "F.Cu") (net 7))
 )
     (attr dnp)
